File: Braille Evaluation Board/Braille Evaluation Board.kicad_pcb (KiCad board)
At the start: 2 copper layers, 90 x 94 mm, 98 parts, among them J101 Conn_01x02, J102 Screw_Terminal_01x02, J103 Conn_01x02, J104 Screw_Terminal_01x02, SW101 SW_Push, SW102 SW_Push, U101 LM317_SOT-223, U102 RP2040-Zero, U201 74HC238, U202 74HC238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

Commit message: Create Rev 1
Parts:
- moved C101 51.1 mm to (92.0, 59.4)
- moved C102 51.1 mm to (102.4, 70.0)
- moved JP101 51.1 mm to (107.9, 60.0)
- moved R101 51.1 mm to (102.5, 64.0)
- moved RV101 51.1 mm to (110.1, 70.5)
- moved U101 51.1 mm to (95.0, 67.0)
- moved U102 44.3 mm to (95.1, 102.2)
- moved D101 16.0 mm to (101.5, 99.0)
- moved D102 16.0 mm to (112.5, 99.0)
- moved R102 16.0 mm to (106.9, 99.0)
- moved R103 15.1 mm to (102.0, 84.0)
- moved J101 12.0 mm to (107.0, 78.5)
- moved J102 12.0 mm to (115.0, 82.0)
- moved J103 12.0 mm to (107.0, 89.5)
- moved J104 12.0 mm to (115.0, 93.0)
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Routing:
- net /DRIVE_CELL_4_LOW: track 0.00 -> 188.5 mm, vias 0 -> 8
- net /MUX_RESET: track 0.00 -> 171.8 mm, vias 0 -> 6
- net /MUX_SET: track 0.00 -> 170.2 mm, vias 0 -> 7
- net Net-(D803-K-Pad3): track 0.00 -> 163.4 mm, vias 0 -> 8
- net /MUX_SELECT_CELL_A2: track 0.00 -> 161.5 mm, vias 0 -> 5
- net /MUX_SELECT_CELL_A1: track 0.00 -> 160.0 mm, vias 0 -> 4
- net /MUX_SELECT_CELL_A0: track 0.00 -> 158.4 mm, vias 0 -> 4
- net +3V3: track 12.9 -> 165.7 mm, vias 0 -> 5
- net Net-(D1003-K-Pad3): track 0.00 -> 147.4 mm, vias 0 -> 6
- net Vdrive: track 16.9 -> 160.8 mm, vias 0 -> 5
- net /DRIVE_CELL_6_HIGH: track 0.00 -> 142.0 mm, vias 0 -> 6
- net /DRIVE_CELL_5_HIGH: track 0.00 -> 138.7 mm, vias 0 -> 8
- net Net-(D702-K-Pad3): track 0.00 -> 137.5 mm, vias 0 -> 6
- net /DRIVE_DOT_6_HIGH: track 0.00 -> 133.3 mm, vias 0 -> 5
- net /DRIVE_DOT_4_HIGH: track 0.00 -> 132.5 mm, vias 0 -> 6
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Other:
- board text added: "GitHub: DeflateAwning ${ISSUE_DATE} ${REVISION}"
