File: Braille Evaluation Board/Braille Evaluation Board.kicad_sch (KiCad schematic)
At the start: 18 parts, among them J101 Conn_01x02, J102 Screw_Terminal_01x02, J103 Conn_01x02, J104 Screw_Terminal_01x02, SW101 SW_Push, SW102 SW_Push, U101 LM317_SOT-223, U102 RP2040-Zero

Commit message: Create Rev 1
Parts:
- D101, D102: footprint Capacitor_SMD:C_1206_3216Metric_Pad1.33x1.80mm_HandSolder -> LED_SMD:LED_1206_3216Metric_Pad1.42x1.75mm_HandSolder
Changed lines of the file:
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@@
 	(generator_version "8.0")
 	(paper "USLetter")
+	(title_block
+		(date "2024-08-30")
+		(rev "Rev 1")
+	)
 	(junction
 		(at 29.21 191.77)
@@
 			)
 		)
-		(property "Footprint" "Capacitor_SMD:C_1206_3216Metric_Pad1.33x1.80mm_HandSolder"
+		(property "Footprint" "LED_SMD:LED_1206_3216Metric_Pad1.42x1.75mm_HandSolder"
 			(at 76.2 177.8 0)
 			(effects
@@
 			)
 		)
-		(property "Footprint" "Capacitor_SMD:C_1206_3216Metric_Pad1.33x1.80mm_HandSolder"
+		(property "Footprint" "LED_SMD:LED_1206_3216Metric_Pad1.42x1.75mm_HandSolder"
 			(at 80.01 177.8 0)
 			(effects
